File: DSP_Hat/DSP_Hat.kicad_pcb (KiCad board)
At the start: 2 copper layers, 65 x 56 mm, 5 parts, among them P1 Conn_02x20_Odd_Even

Commit message: farted around some more with DSP Hat
Parts:
- added R2: 2k, Resistor_SMD:R_0402_1005Metric, F.Cu at (237.3, 115.7)
- added R3: 2k, Resistor_SMD:R_0402_1005Metric, F.Cu at (241.9, 115.7)
- added R4: 49.9, Resistor_SMD:R_0402_1005Metric, F.Cu at (227.5, 113.2)
- added R5: 10k, Resistor_SMD:R_0402_1005Metric, F.Cu at (215.2, 135.5)
- added U1: ADAU1761BCPZ-R7, DSP_Hat:ADAU1761BCPZ-R7, F.Cu at (249.5, 114.4)
- added X1: 25MHz, Oscillator:Oscillator_SMD_Abracon_ASV-4Pin_7.0x5.1mm, F.Cu at (224.1, 136.0)

Commit message: overhaul of schematic
Parts:
- added C1: 10uF, Capacitor_SMD:C_0805_2012Metric_Pad1.15x1.40mm_HandSolder, F.Cu at (230.5, 114.4)
- added C10: 0.1uF, Capacitor_SMD:C_0603_1608Metric_Pad1.05x0.95mm_HandSolder, F.Cu at (236.8, 104.3)
- added C11: 0.1uF, Capacitor_SMD:C_0603_1608Metric_Pad1.05x0.95mm_HandSolder, F.Cu at (212.7, 120.4)
- added C12: 10uF, Capacitor_SMD:C_0805_2012Metric_Pad1.15x1.40mm_HandSolder, F.Cu at (216.3, 120.5)
- added C13: 9.1 pF, Capacitor_SMD:C_0603_1608Metric_Pad1.05x0.95mm_HandSolder, F.Cu at (254.2, 129.7)
- added C2: 10uF, Capacitor_SMD:C_0805_2012Metric_Pad1.15x1.40mm_HandSolder, F.Cu at (253.1, 122.1)
- added C3: 0.1uF, Capacitor_SMD:C_0603_1608Metric_Pad1.05x0.95mm_HandSolder, F.Cu at (253.7, 134.8)
- added C4: 0.1uF, Capacitor_SMD:C_0603_1608Metric_Pad1.05x0.95mm_HandSolder, F.Cu at (253.7, 139.8)
- added C5: 0.1uF, Capacitor_SMD:C_0603_1608Metric_Pad1.05x0.95mm_HandSolder, F.Cu at (253.7, 132.2)
- added C6: 10uf, Capacitor_SMD:C_0805_2012Metric_Pad1.15x1.40mm_HandSolder, F.Cu at (217.5, 109.4)
- added C7: 10uf, Capacitor_SMD:C_0805_2012Metric_Pad1.15x1.40mm_HandSolder, F.Cu at (217.5, 134.8)
- added C8: 10uf, Capacitor_SMD:C_0805_2012Metric_Pad1.15x1.40mm_HandSolder, F.Cu at (217.5, 139.8)
- added C9: 10uf, Capacitor_SMD:C_0805_2012Metric_Pad1.15x1.40mm_HandSolder, F.Cu at (218.0, 104.3)
- added J1: Screw_Terminal_01x02, TerminalBlock:TerminalBlock_Altech_AK300-2_P5.00mm, F.Cu at (208.9, 109.4)
- added J2: Screw_Terminal_01x02, TerminalBlock:TerminalBlock_Altech_AK300-2_P5.00mm, F.Cu at (208.9, 139.8)
- added L2: L_Core_Ferrite, Inductor_SMD:L_0402_1005Metric, F.Cu at (240.2, 115.7)
- R4: footprint Resistor_SMD:R_0402_1005Metric -> Resistor_SMD:R_0603_1608Metric
- moved R5 38.6 mm to (233.0, 101.3), turned to 180 degrees
- moved R3 35.7 mm to (208.9, 129.2), turned to 270 degrees
- moved X1 29.5 mm to (231.8, 107.5), turned to 270 degrees
- moved R2 28.5 mm to (208.9, 114.4), turned to 270 degrees
- moved U1 23.4 mm to (226.7, 119.5), turned to 180 degrees
- moved R4 10.5 mm to (237.6, 110.6)

Commit message: I hate working with KiCad symbol and footprint libraries
Parts:
- added FER1: 600, Inductor_SMD:L_0603_1608Metric_Pad1.05x0.95mm_HandSolder, F.Cu at (257.7, 110.1)
- added R1: 10K, Resistor_SMD:R_0603_1608Metric_Pad1.05x0.95mm_HandSolder, F.Cu at (257.7, 111.6)
- added R10: 100K, Resistor_SMD:R_0402_1005Metric, F.Cu at (260.3, 110.8)
- added R6: 470.0K, Resistor_SMD:R_0402_1005Metric, F.Cu at (260.3, 109.9)
- added R9: 100K, Resistor_SMD:R_0402_1005Metric, F.Cu at (257.0, 112.9)
- added Y1: ASFLMB-12.288MHZ-LC-T_0, DSP_Hat:ASFLMB-12.288MHZ-LC-T, F.Cu at (254.1, 112.2)
- C10, C3, C5: value 0.1uF -> 10uF
- C11: value 0.1uF -> 100uF
- C12: value 10uF -> 0.1 uF
- C13: value 9.1 pF -> 0.1 uF
- C6, C7: value 10uf -> 0.1uF
- C8: value 10uf -> 10uF
- C9: value 10uf -> 100uF
- J1, J2: value Screw_Terminal_01x02 -> AudioJack2_Ground_Switch
- R2: value 2k -> 10K
- R3: value 2k -> 100K
- R4: value 49.9 -> 100K
- R5: value 10k -> 470.0K
- U1: value ADAU1761BCPZ-R7 -> ADAU1761BCPZ-R7_2
Connections:
- net Net-(U1-Pad15) renamed /ROUTP
- net Net-(U1-Pad16) renamed /ROUTN
- net Net-(U1-Pad17) renamed /LOUTN
- net Net-(U1-Pad18) renamed /LOUTP
- net Net-(U1-Pad26) renamed /ADC_SDATA
- net Net-(U1-Pad27) renamed /DAC_SDATA
- net Net-(U1-Pad29) renamed /LRCLK
- net Net-(U1-Pad3) renamed /ADAIU761_ADDR0
- net Net-(U1-Pad30) renamed /ADAIU761_ADDR1
- net Net-(U1-Pad31) renamed /TWIO_SDA
- net Net-(U1-Pad32) renamed /TWI0_SCL
- C1 pad 1: +3V3 -> Net-(C1-Pad1)
- C1 pad 2: GND -> Net-(C1-Pad2)
- C10 pad 1: GND -> Net-(C10-Pad1)
- C10 pad 2: Net-(C10-Pad2) -> GND
- C11 pad 2: GND -> Net-(C11-Pad2)
- C12 pad 1: Net-(C11-Pad1) -> Net-(C10-Pad1)
- C13 pad 1: Net-(C13-Pad1) -> Net-(C10-Pad1)
- C2 pad 1: +3V3 -> Net-(C2-Pad1)
- C2 pad 2: GND -> Net-(C2-Pad2)
- C5 pad 1: +3V3 -> Net-(C5-Pad1)
- C6 pad 1: /LINN -> Net-(C5-Pad1)
- C6 pad 2: Net-(C6-Pad2) -> GND
- C7 pad 1: /RINN -> GND
- C8 pad 1: /RINP -> GND
- C8 pad 2: GND -> Net-(C7-Pad2)
- C9 pad 1: /LINP -> Net-(C9-Pad1)
- C9 pad 2: GND -> Net-(C9-Pad2)
- J1 pad 1: Net-(C6-Pad2) -> (no net)
- J1 pad 2: GND -> (no net)
- J2 pad 1: GND -> (no net)
- J2 pad 2: Net-(C7-Pad2) -> (no net)
- R2 pad 1: Net-(C6-Pad2) -> Net-(R1-Pad2)
- R2 pad 2: /MICBIAS -> GND
- R3 pad 1: /MICBIAS -> GND
- R3 pad 2: Net-(C7-Pad2) -> Net-(C2-Pad2)
- R4 pad 1: Net-(R4-Pad1) -> GND
- R4 pad 2: /MCLK -> Net-(C1-Pad2)
- R5 pad 1: Net-(C10-Pad2) -> GND
- R5 pad 2: Net-(R5-Pad2) -> Net-(C2-Pad1)
- U1 pad 10: /LINP -> Net-(C7-Pad2)
- U1 pad 11: /LINN -> Net-(C1-Pad1)
- U1 pad 12: /RINP -> Net-(C7-Pad2)
- U1 pad 13: /RINN -> Net-(C2-Pad1)
- U1 pad 14: Net-(U1-Pad14) -> Net-(C7-Pad2)
- U1 pad 19: Net-(U1-Pad19) -> Net-(C11-Pad1)
- U1 pad 2: /MCLK -> Net-(R7-Pad2)
- U1 pad 20: Net-(U1-Pad20) -> Net-(C9-Pad1)
- U1 pad 23: +3V3 -> Net-(C10-Pad1)
- U1 pad 24: Net-(C11-Pad1) -> Net-(C5-Pad1)
- U1 pad 33: Net-(U1-Pad33) -> GND
- U1 pad 4: Net-(U1-Pad4) -> Net-(C7-Pad2)
- U1 pad 5: /MICBIAS -> Net-(U1-Pad5)
- U1 pad 6: Net-(U1-Pad6) -> Net-(C7-Pad2)
- U1 pad 7: Net-(U1-Pad7) -> Net-(C7-Pad2)
- U1 pad 8: +3V3 -> Net-(C10-Pad1)
