File: DSP_Hat/DSP_Hat.sch (KiCad schematic (older format))
At the start: 35 parts, among them P1 Conn_02x20_Odd_Even

Commit message: annotate parts
Parts:
- gave numbers to parts that had none: 30

Commit message: associating footprints to symbols
Parts:
- R1, R2: footprint (none) -> Resistor_SMD:R_0603_1608Metric_Pad1.05x0.95mm_HandSolder
Changed lines of the file:
@@
 F 0 "R1" H 1970 5546 50  0000 L CNN
 F 1 "10K" H 1970 5455 50  0000 L CNN
-F 2 "" V 1830 5500 50  0001 C CNN
+F 2 "Resistor_SMD:R_0603_1608Metric_Pad1.05x0.95mm_HandSolder" V 1830 5500 50  0001 C CNN
 F 3 "~" H 1900 5500 50  0001 C CNN
 	1    1900 5500
@@
 F 0 "R2" H 1970 5946 50  0000 L CNN
 F 1 "10K" H 1970 5855 50  0000 L CNN
-F 2 "" V 1830 5900 50  0001 C CNN
+F 2 "Resistor_SMD:R_0603_1608Metric_Pad1.05x0.95mm_HandSolder" V 1830 5900 50  0001 C CNN
 F 3 "~" H 1900 5900 50  0001 C CNN
 	1    1900 5900

Commit message: futher matching of footprints to symbols
Parts:
- C1, C10, C2, C3, C5: footprint (none) -> Capacitor_SMD:C_0805_2012Metric_Pad1.15x1.40mm_HandSolder
- C12, C13, C4, C6, C7, C8: footprint (none) -> Capacitor_SMD:C_0603_1608Metric_Pad1.05x0.95mm_HandSolder
- FER1: footprint (none) -> Inductor_SMD:L_0603_1608Metric_Pad1.05x0.95mm_HandSolder
- R10, R3, R4, R5, R6, R9: footprint (none) -> Resistor_SMD:R_0402_1005Metric
- U1: footprint CP_32_4 -> (none)
- Y1: footprint ASFLMB_Series -> (none)
Changed lines of the file:
@@
 F 0 "U1" H 7800 2987 60  0000 C CNN
 F 1 "ADAU1761BCPZ-R7_2" H 7800 2881 60  0000 C CNN
-F 2 "CP_32_4" H 7750 2890 60  0001 C CNN
+F 2 "" H 7750 2890 60  0001 C CNN
 F 3 "" H 6000 2450 60  0000 C CNN
 	1    7100 2800
@@
 F 0 "FER1" V 8322 2050 50  0000 C CNN
 F 1 "600" V 8413 2050 50  0000 C CNN
-F 2 "" H 8500 2050 50  0001 C CNN
+F 2 "Inductor_SMD:L_0603_1608Metric_Pad1.05x0.95mm_HandSolder" H 8500 2050 50  0001 C CNN
 F 3 "~" H 8500 2050 50  0001 C CNN
 	1    8500 2050
@@
 F 0 "R3" H 3519 4504 50  0000 L CNN
 F 1 "100K" H 3519 4595 50  0000 L CNN
-F 2 "" V 3380 4550 50  0001 C CNN
+F 2 "Resistor_SMD:R_0402_1005Metric" V 3380 4550 50  0001 C CNN
 F 3 "~" H 3450 4550 50  0001 C CNN
 	1    3450 4550
@@
 F 0 "R4" H 3630 4504 50  0000 R CNN
 F 1 "100K" H 3630 4595 50  0000 R CNN
-F 2 "" V 3630 4550 50  0001 C CNN
+F 2 "Resistor_SMD:R_0402_1005Metric" V 3630 4550 50  0001 C CNN
 F 3 "~" H 3700 4550 50  0001 C CNN
 	1    3700 4550
@@
 F 0 "R5" H 4820 4504 50  0000 L CNN
 F 1 "470.0K" H 4820 4595 50  0000 L CNN
-F 2 "" V 4680 4550 50  0001 C CNN
+F 2 "Resistor_SMD:R_0402_1005Metric" V 4680 4550 50  0001 C CNN
 F 3 "~" H 4750 4550 50  0001 C CNN
 	1    4750 4550
@@
 F 0 "R6" H 4930 4504 50  0000 R CNN
 F 1 "470.0K" H 4930 4595 50  0000 R CNN
-F 2 "" V 4930 4550 50  0001 C CNN
+F 2 "Resistor_SMD:R_0402_1005Metric" V 4930 4550 50  0001 C CNN
 F 3 "~" H 5000 4550 50  0001 C CNN
 	1    5000 4550
@@
 F 0 "R10" H 9630 3904 50  0000 R CNN
 F 1 "100K" H 9630 3995 50  0000 R CNN
-F 2 "" V 9630 3950 50  0001 C CNN
+F 2 "Resistor_SMD:R_0402_1005Metric" V 9630 3950 50  0001 C CNN
 F 3 "~" H 9700 3950 50  0001 C CNN
 	1    9700 3950
@@
 F 0 "R9" H 9230 3904 50  0000 R CNN
 F 1 "100K" H 9230 3995 50  0000 R CNN
-F 2 "" V 9230 3950 50  0001 C CNN
+F 2 "Resistor_SMD:R_0402_1005Metric" V 9230 3950 50  0001 C CNN
 F 3 "~" H 9300 3950 50  0001 C CNN
 	1    9300 3950
@@
 F 0 "C3" H 4692 2946 50  0000 L CNN
 F 1 "10uF" H 4692 2855 50  0000 L CNN
-F 2 "" H 4600 2900 50  0001 C CNN
+F 2 "Capacitor_SMD:C_0805_2012Metric_Pad1.15x1.40mm_HandSolder" H 4600 2900 50  0001 C CNN
 F 3 "~" H 4600 2900 50  0001 C CNN
 	1    4600 2900
@@
 F 0 "C4" H 5192 2946 50  0000 L CNN
 F 1 "0.1uF" H 5192 2855 50  0000 L CNN
-F 2 "" H 5100 2900 50  0001 C CNN
+F 2 "Capacitor_SMD:C_0603_1608Metric_Pad1.05x0.95mm_HandSolder" H 5100 2900 50  0001 C CNN
 F 3 "~" H 5100 2900 50  0001 C CNN
 	1    5100 2900
@@
 F 0 "C5" H 5692 2946 50  0000 L CNN
 F 1 "10uF" H 5692 2855 50  0000 L CNN
-F 2 "" H 5600 2900 50  0001 C CNN
+F 2 "Capacitor_SMD:C_0805_2012Metric_Pad1.15x1.40mm_HandSolder" H 5600 2900 50  0001 C CNN
 F 3 "~" H 5600 2900 50  0001 C CNN
 	1    5600 2900
@@
 F 0 "C6" H 6142 2946 50  0000 L CNN
 F 1 "0.1uF" H 6142 2855 50  0000 L CNN
-F 2 "" H 6050 2900 50  0001 C CNN
+F 2 "Capacitor_SMD:C_0603_1608Metric_Pad1.05x0.95mm_HandSolder" H 6050 2900 50  0001 C CNN
 F 3 "~" H 6050 2900 50  0001 C CNN
 	1    6050 2900
@@
 F 0 "C13" H 10542 2296 50  0000 L CNN
 F 1 "0.1 uF" H 10542 2205 50  0000 L CNN
-F 2 "" H 10450 2250 50  0001 C CNN
+F 2 "Capacitor_SMD:C_0603_1608Metric_Pad1.05x0.95mm_HandSolder" H 10450 2250 50  0001 C CNN
 F 3 "~" H 10450 2250 50  0001 C CNN
 	1    10450 2250
@@
 F 0 "C12" H 10042 2296 50  0000 L CNN
 F 1 "0.1 uF" H 10042 2205 50  0000 L CNN
-F 2 "" H 9950 2250 50  0001 C CNN
+F 2 "Capacitor_SMD:C_0603_1608Metric_Pad1.05x0.95mm_HandSolder" H 9950 2250 50  0001 C CNN
 F 3 "~" H 9950 2250 50  0001 C CNN
 	1    9950 2250
@@
 F 0 "C10" H 9442 2296 50  0000 L CNN
 F 1 "10uF" H 9442 2205 50  0000 L CNN
-F 2 "" H 9350 2250 50  0001 C CNN
+F 2 "Capacitor_SMD:C_0805_2012Metric_Pad1.15x1.40mm_HandSolder" H 9350 2250 50  0001 C CNN
 F 3 "~" H 9350 2250 50  0001 C CNN
 	1    9350 2250
@@
 F 0 "C1" V 3821 4050 50  0000 C CNN
 F 1 "10uF" V 3912 4050 50  0000 C CNN
-F 2 "" H 4050 4050 50  0001 C CNN
+F 2 "Capacitor_SMD:C_0805_2012Metric_Pad1.15x1.40mm_HandSolder" H 4050 4050 50  0001 C CNN
 F 3 "~" H 4050 4050 50  0001 C CNN
 	1    4050 4050
@@
 F 0 "C2" V 4437 4250 50  0000 C CNN
 F 1 "10uF" V 4528 4250 50  0000 C CNN
-F 2 "" H 4300 4250 50  0001 C CNN
+F 2 "Capacitor_SMD:C_0805_2012Metric_Pad1.15x1.40mm_HandSolder" H 4300 4250 50  0001 C CNN
 F 3 "~" H 4300 4250 50  0001 C CNN
 	1    4300 4250
@@
 F 0 "C7" H 6341 6154 50  0000 L CNN
 F 1 "0.1uF" H 6341 6245 50  0000 L CNN
-F 2 "" H 6250 6200 50  0001 C CNN
+F 2 "Capacitor_SMD:C_0603_1608Metric_Pad1.05x0.95mm_HandSolder" H 6250 6200 50  0001 C CNN
 F 3 "~" H 6250 6200 50  0001 C CNN
 	1    6250 6200
@@
 F 0 "C8" H 6458 6154 50  0000 R CNN
 F 1 "10uF" H 6458 6245 50  0000 R CNN
-F 2 "" H 6550 6200 50  0001 C CNN
+F 2 "Capacitor_SMD:C_0603_1608Metric_Pad1.05x0.95mm_HandSolder" H 6550 6200 50  0001 C CNN
 F 3 "~" H 6550 6200 50  0001 C CNN
 	1    6550 6200
@@
 F 0 "Y1" H 3175 6087 60  0000 C CNN
 F 1 "ASFLMB-12.288MHZ-LC-T_0" H 3175 5981 60  0000 C CNN
-F 2 "ASFLMB_Series" H 3150 5950 60  0001 C CNN
+F 2 "" H 3150 5950 60  0001 C CNN
 F 3 "" H 2500 5700 60  0000 C CNN
 	1    2500 5700

Commit message: corrected path for missing library
Parts:
- U1: footprint (none) -> DSP_Hat:ADAU1761BCPZ-R7
- Y1: footprint (none) -> DSP_Hat:ASFLMB-12.288MHZ-LC-T
Changed lines of the file:
@@
 F 0 "U1" H 7800 2987 60  0000 C CNN
 F 1 "ADAU1761BCPZ-R7_2" H 7800 2881 60  0000 C CNN
-F 2 "" H 7750 2890 60  0001 C CNN
+F 2 "DSP_Hat:ADAU1761BCPZ-R7" H 7750 2890 60  0001 C CNN
 F 3 "" H 6000 2450 60  0000 C CNN
 	1    7100 2800
@@
 F 0 "Y1" H 3175 6087 60  0000 C CNN
 F 1 "ASFLMB-12.288MHZ-LC-T_0" H 3175 5981 60  0000 C CNN
-F 2 "" H 3150 5950 60  0001 C CNN
+F 2 "DSP_Hat:ASFLMB-12.288MHZ-LC-T" H 3150 5950 60  0001 C CNN
 F 3 "" H 2500 5700 60  0000 C CNN
 	1    2500 5700

Commit message: I hate working with KiCad symbol and footprint libraries
Parts:
- C11, C9: footprint (none) -> DSP_Hat:UWX1C101MCL1GB
Changed lines of the file:
@@
 F 0 "C9" V 9355 3600 50  0000 C CNN
 F 1 "100uF" V 9264 3600 50  0000 C CNN
-F 2 "" H 9138 3450 50  0001 C CNN
+F 2 "DSP_Hat:UWX1C101MCL1GB" H 9138 3450 50  0001 C CNN
 F 3 "~" H 9100 3600 50  0001 C CNN
 	1    9100 3600
@@
 F 0 "C11" V 9755 3700 50  0000 C CNN
 F 1 "100uF" V 9664 3700 50  0000 C CNN
-F 2 "" H 9538 3550 50  0001 C CNN
+F 2 "DSP_Hat:UWX1C101MCL1GB" H 9538 3550 50  0001 C CNN
 F 3 "~" H 9500 3700 50  0001 C CNN
 	1    9500 3700
